File: Hardware/V1/V1.sch (KiCad schematic (older format))
At the start: 68 parts, among them J1 Conn_01x03, J2 Conn_Coaxial, J3 USB_B_Micro, J4 Encoder, J5 Conn_01x10, Q1 MMSS8050-H-TP, Q2 MMSS8050-H-TP, U1 AMS1117-3.3, U2 ADS8689IPW, U3 CP2102N-A01-GQFN24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

Commit message: changed 100n to 0.1u
Parts:
- C13, C17, C19, C21, C22, C23, C25, C26, C27, C5: value 100nF -> 0.1uF
Changed lines of the file:
@@
 P 7850 3150
 F 0 "C17" H 7965 3196 50  0000 L CNN
-F 1 "100nF" H 7965 3105 50  0000 L CNN
+F 1 "0.1uF" H 7965 3105 50  0000 L CNN
 F 2 "digikey-footprints:0603" H 7888 3000 50  0001 C CNN
 F 3 "~" H 7850 3150 50  0001 C CNN
@@
 P 2450 2950
 F 0 "C13" H 2565 2996 50  0000 L CNN
-F 1 "100nF" H 2565 2905 50  0000 L CNN
+F 1 "0.1uF" H 2565 2905 50  0000 L CNN
 F 2 "digikey-footprints:0603" H 2488 2800 50  0001 C CNN
 F 3 "~" H 2450 2950 50  0001 C CNN
@@
 P 2750 1750
 F 0 "C5" H 2865 1796 50  0000 L CNN
-F 1 "100nF" H 2865 1705 50  0000 L CNN
+F 1 "0.1uF" H 2865 1705 50  0000 L CNN
 F 2 "digikey-footprints:0603" H 2788 1600 50  0001 C CNN
 F 3 "~" H 2750 1750 50  0001 C CNN
@@
 P 10850 3200
 F 0 "C21" H 10886 3324 50  0000 L CNN
-F 1 "100nF" H 10887 3115 50  0000 L CNN
+F 1 "0.1uF" H 10887 3115 50  0000 L CNN
 F 2 "digikey-footprints:0603" H 10888 3050 50  0001 C CNN
 F 3 "~" H 10850 3200 50  0001 C CNN
@@
 P 13150 3150
 F 0 "C19" H 13186 3274 50  0000 L CNN
-F 1 "100nF" H 13187 3065 50  0000 L CNN
+F 1 "0.1uF" H 13187 3065 50  0000 L CNN
 F 2 "digikey-footprints:0603" H 13188 3000 50  0001 C CNN
 F 3 "~" H 13150 3150 50  0001 C CNN
@@
 P 14650 3600
 F 0 "C22" H 14765 3646 50  0000 L CNN
-F 1 "100nF" H 14765 3555 50  0000 L CNN
+F 1 "0.1uF" H 14765 3555 50  0000 L CNN
 F 2 "digikey-footprints:0603" H 14688 3450 50  0001 C CNN
 F 3 "~" H 14650 3600 50  0001 C CNN
@@
 AR Path="/614B6C0E" Ref="C25"  Part="1"
 F 0 "C25" H 5965 6646 50  0000 L CNN
-F 1 "100nF" H 5965 6555 50  0000 L CNN
+F 1 "0.1uF" H 5965 6555 50  0000 L CNN
 F 2 "digikey-footprints:0603" H 5888 6450 50  0001 C CNN
 F 3 "~" H 5850 6600 50  0001 C CNN
@@
 P 5200 8000
 F 0 "C26" H 5315 8046 50  0000 L CNN
-F 1 "100nF" H 5315 7955 50  0000 L CNN
+F 1 "0.1uF" H 5315 7955 50  0000 L CNN
 F 2 "digikey-footprints:0603" H 5238 7850 50  0001 C CNN
 F 3 "~" H 5200 8000 50  0001 C CNN
@@
 P 3200 3200
 F 0 "C23" H 3315 3246 50  0000 L CNN
-F 1 "100nF" H 3315 3155 50  0000 L CNN
+F 1 "0.1uF" H 3315 3155 50  0000 L CNN
 F 2 "digikey-footprints:0603" H 3238 3050 50  0001 C CNN
 F 3 "~" H 3200 3200 50  0001 C CNN
@@
 P 14750 2300
 F 0 "C27" H 14786 2424 50  0000 L CNN
-F 1 "100nF" H 14787 2215 50  0000 L CNN
+F 1 "0.1uF" H 14787 2215 50  0000 L CNN
 F 2 "digikey-footprints:0603" H 14788 2150 50  0001 C CNN
 F 3 "~" H 14750 2300 50  0001 C CNN
